File: kicad/eepromcape.kicad_pcb (KiCad board)
At the start: 2 copper layers, 33 x 22.9 mm, 5 parts, among them J1 Conn_01x12, J2 Conn_01x12, J3 Conn_02x04_Counter_Clockwise

Commit message: Update eepromcape.kicad_pcb
Parts:
- renumbered J2 to 3.3, J3 to TC, J1 to VB
Routing:
- net GND: vias 35 -> 43
Other:
- board text added: "G"
Changed lines of the file:
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@@
   (general
     (thickness 1.6)
-    (drawings 12)
-    (tracks 54)
+    (drawings 13)
+    (tracks 62)
     (zones 0)
     (modules 5)
@@
     (mod_text_size 1 1)
     (mod_text_width 0.15)
-    (pad_size 1.524 1.524)
-    (pad_drill 0.762)
+    (pad_size 1 1)
+    (pad_drill 0)
     (pad_to_mask_clearance 0)
     (aux_axis_origin 0 0)
@@
     (descr "Through hole straight socket strip, 2x04, 2.54mm pitch, double cols (from Kicad 4.0.7), script generated")
     (tags "Through hole socket strip THT 2x04 2.54mm double row")
-    (fp_text reference J3 (at -1.27 2.77 270) (layer F.SilkS)
+    (fp_text reference TC (at -1.27 2.77 270) (layer F.SilkS)
       (effects (font (size 1 1) (thickness 0.15)))
     )
@@
     (descr "Through hole straight pin header, 1x12, 2.54mm pitch, single row")
     (tags "Through hole pin header THT 1x12 2.54mm single row")
-    (fp_text reference J1 (at -2.54 -0.010201 90) (layer F.SilkS)
+    (fp_text reference VB (at -2.54 -0.010201 90) (layer F.SilkS)
       (effects (font (size 1 1) (thickness 0.15)))
     )
@@
     (descr "Through hole straight pin header, 1x12, 2.54mm pitch, single row")
     (tags "Through hole pin header THT 1x12 2.54mm single row")
-    (fp_text reference J2 (at 2.54 -0.010201 90) (layer F.SilkS)
+    (fp_text reference 3.3 (at 2.54 -0.010201 90) (layer F.SilkS)
       (effects (font (size 1 1) (thickness 0.15)))
     )
@@
     )
   )
+  (gr_text G (at 88.9 65.786 90) (layer F.SilkS)
+    (effects (font (size 1 1) (thickness 0.15)) (justify left))
+  )
   (gr_text DO (at 114.3 86.106 90) (layer F.SilkS)
     (effects (font (size 1 1) (thickness 0.15)) (justify left))
@@
   (gr_line (start 115.580201 86.36) (end 85.100201 86.36) (layer Edge.Cuts) (width 0.1))
   (segment (start 106.690201 75.776667) (end 106.690201 82.55) (width 0.635) (layer F.Cu) (net 21))
+  (segment (start 99.0652 75.776667) (end 106.690201 75.776667) (width 0.635) (layer B.Cu) (net 21))
   (segment (start 96.5252 73.236667) (end 99.0652 75.776667) (width 0.635) (layer B.Cu) (net 21))
-  (segment (start 99.0652 75.776667) (end 106.690201 75.776667) (width 0.635) (layer B.Cu) (net 21))
   (segment (start 109.230201 75.776667) (end 109.230201 82.55) (width 0.635) (layer F.Cu) (net 22))
   (segment (start 111.770201 75.776667) (end 111.770201 82.55) (width 0.635) (layer F.Cu) (net 23))
@@
   (segment (start 94.0152 75.77) (end 97.2052 78.96) (width 0.635) (layer B.Cu) (net 24))
   (segment (start 88.9052 67.315001) (end 88.910201 67.31) (width 1.016) (layer B.Cu) (net 25))
-  (via (at 86.36 65.024) (size 0.8) (drill 0.4) (layers F.Cu B.Cu) (net 25))
-  (via (at 88.9 65.024) (size 0.8) (drill 0.4) (layers F.Cu B.Cu) (net 25))
-  (via (at 91.44 65.024) (size 0.8) (drill 0.4) (layers F.Cu B.Cu) (net 25))
-  (via (at 93.98 65.024) (size 0.8) (drill 0.4) (layers F.Cu B.Cu) (net 25))
-  (via (at 96.52 65.024) (size 0.8) (drill 0.4) (layers F.Cu B.Cu) (net 25))
-  (via (at 99.06 65.024) (size 0.8) (drill 0.4) (layers F.Cu B.Cu) (net 25))
-  (via (at 101.6 65.024) (size 0.8) (drill 0.4) (layers F.Cu B.Cu) (net 25))
-  (via (at 104.14 65.024) (size 0.8) (drill 0.4) (layers F.Cu B.Cu) (net 25))
-  (via (at 106.68 65.024) (size 0.8) (drill 0.4) (layers F.Cu B.Cu) (net 25))
-  (via (at 109.22 65.024) (size 0.8) (drill 0.4) (layers F.Cu B.Cu) (net 25))
-  (via (at 111.76 65.024) (size 0.8) (drill 0.4) (layers F.Cu B.Cu) (net 25))
-  (via (at 114.3 65.024) (size 0.8) (drill 0.4) (layers F.Cu B.Cu) (net 25))
-  (via (at 86.36 84.836) (size 0.8) (drill 0.4) (layers F.Cu B.Cu) (net 25))
-  (via (at 88.9 84.836) (size 0.8) (drill 0.4) (layers F.Cu B.Cu) (net 25))
-  (via (at 91.44 84.836) (size 0.8) (drill 0.4) (layers F.Cu B.Cu) (net 25))
-  (via (at 93.98 84.836) (size 0.8) (drill 0.4) (layers F.Cu B.Cu) (net 25))
-  (via (at 96.52 84.836) (size 0.8) (drill 0.4) (layers F.Cu B.Cu) (net 25))
-  (via (at 99.06 84.836) (size 0.8) (drill 0.4) (layers F.Cu B.Cu) (net 25))
-  (via (at 101.6 84.836) (size 0.8) (drill 0.4) (layers F.Cu B.Cu) (net 25))
-  (via (at 104.14 84.836) (size 0.8) (drill 0.4) (layers F.Cu B.Cu) (net 25))
-  (via (at 106.68 84.836) (size 0.8) (drill 0.4) (layers F.Cu B.Cu) (net 25))
-  (via (at 109.22 84.836) (size 0.8) (drill 0.4) (layers F.Cu B.Cu) (net 25))
-  (via (at 111.76 84.836) (size 0.8) (drill 0.4) (layers F.Cu B.Cu) (net 25))
-  (via (at 114.3 84.836) (size 0.8) (drill 0.4) (layers F.Cu B.Cu) (net 25))
-  (via (at 106.68 70.358) (size 0.8) (drill 0.4) (layers F.Cu B.Cu) (net 25))
-  (via (at 109.22 70.358) (size 0.8) (drill 0.4) (layers F.Cu B.Cu) (net 25))
-  (via (at 111.76 70.358) (size 0.8) (drill 0.4) (layers F.Cu B.Cu) (net 25))
-  (via (at 114.3 70.358) (size 0.8) (drill 0.4) (layers F.Cu B.Cu) (net 25))
-  (via (at 103.886 73.152) (size 0.8) (drill 0.4) (layers F.Cu B.Cu) (net 25))
-  (via (at 101.6 73.152) (size 0.8) (drill 0.4) (layers F.Cu B.Cu) (net 25))
-  (via (at 99.06 73.152) (size 0.8) (drill 0.4) (layers F.Cu B.Cu) (net 25))
-  (via (at 86.36 79.248) (size 0.8) (drill 0.4) (layers F.Cu B.Cu) (net 25))
-  (via (at 88.9 79.248) (size 0.8) (drill 0.4) (layers F.Cu B.Cu) (net 25))
-  (via (at 91.44 79.248) (size 0.8) (drill 0.4) (layers F.Cu B.Cu) (net 25))
-  (via (at 93.98 79.248) (size 0.8) (drill 0.4) (layers F.Cu B.Cu) (net 25))
+  (via (at 85.09 65.024) (size 0.8) (drill 0.4) (layers F.Cu B.Cu) (net 25))
+  (via (at 87.63 65.024) (size 0.8) (drill 0.4) (layers F.Cu B.Cu) (net 25))
+  (via (at 90.17 65.024) (size 0.8) (drill 0.4) (layers F.Cu B.Cu) (net 25))
+  (via (at 92.71 65.024) (size 0.8) (drill 0.4) (layers F.Cu B.Cu) (net 25))
+  (via (at 95.25 65.024) (size 0.8) (drill 0.4) (layers F.Cu B.Cu) (net 25))
+  (via (at 97.79 65.024) (size 0.8) (drill 0.4) (layers F.Cu B.Cu) (net 25))
+  (via (at 100.33 65.024) (size 0.8) (drill 0.4) (layers F.Cu B.Cu) (net 25))
+  (via (at 102.87 65.024) (size 0.8) (drill 0.4) (layers F.Cu B.Cu) (net 25))
+  (via (at 105.41 65.024) (size 0.8) (drill 0.4) (layers F.Cu B.Cu) (net 25))
+  (via (at 107.95 65.024) (size 0.8) (drill 0.4) (layers F.Cu B.Cu) (net 25))
+  (via (at 110.49 65.024) (size 0.8) (drill 0.4) (layers F.Cu B.Cu) (net 25))
+  (via (at 113.03 65.024) (size 0.8) (drill 0.4) (layers F.Cu B.Cu) (net 25))
+  (via (at 85.09 84.836) (size 0.8) (drill 0.4) (layers F.Cu B.Cu) (net 25))
+  (via (at 87.63 84.836) (size 0.8) (drill 0.4) (layers F.Cu B.Cu) (net 25))
+  (via (at 90.17 84.836) (size 0.8) (drill 0.4) (layers F.Cu B.Cu) (net 25))
+  (via (at 92.71 84.836) (size 0.8) (drill 0.4) (layers F.Cu B.Cu) (net 25))
+  (via (at 95.25 84.836) (size 0.8) (drill 0.4) (layers F.Cu B.Cu) (net 25))
+  (via (at 97.79 84.836) (size 0.8) (drill 0.4) (layers F.Cu B.Cu) (net 25))
+  (via (at 100.33 84.836) (size 0.8) (drill 0.4) (layers F.Cu B.Cu) (net 25))
+  (via (at 102.87 84.836) (size 0.8) (drill 0.4) (layers F.Cu B.Cu) (net 25))
+  (via (at 105.41 84.836) (size 0.8) (drill 0.4) (layers F.Cu B.Cu) (net 25))
+  (via (at 107.95 84.836) (size 0.8) (drill 0.4) (layers F.Cu B.Cu) (net 25))
+  (via (at 110.49 84.836) (size 0.8) (drill 0.4) (layers F.Cu B.Cu) (net 25))
+  (via (at 113.03 84.836) (size 0.8) (drill 0.4) (layers F.Cu B.Cu) (net 25))
+  (via (at 105.664 69.596) (size 0.8) (drill 0.4) (layers F.Cu B.Cu) (net 25))
+  (via (at 107.95 71.12) (size 0.8) (drill 0.4) (layers F.Cu B.Cu) (net 25))
+  (via (at 110.49 69.596) (size 0.8) (drill 0.4) (layers F.Cu B.Cu) (net 25))
+  (via (at 113.03 71.12) (size 0.8) (drill 0.4) (layers F.Cu B.Cu) (net 25))
+  (via (at 101.6 74.422) (size 0.8) (drill 0.4) (layers F.Cu B.Cu) (net 25))
+  (via (at 99.06 72.39) (size 0.8) (drill 0.4) (layers F.Cu B.Cu) (net 25))
+  (via (at 87.63 77.978) (size 0.8) (drill 0.4) (layers F.Cu B.Cu) (net 25))
+  (via (at 90.17 80.01) (size 0.8) (drill 0.4) (layers F.Cu B.Cu) (net 25))
+  (via (at 92.71 77.978) (size 0.8) (drill 0.4) (layers F.Cu B.Cu) (net 25))
+  (via (at 95.25 80.01) (size 0.8) (drill 0.4) (layers F.Cu B.Cu) (net 25))
+  (via (at 115.57 65.024) (size 0.8) (drill 0.4) (layers F.Cu B.Cu) (net 25))
+  (via (at 115.57 84.836) (size 0.8) (drill 0.4) (layers F.Cu B.Cu) (net 25))
+  (via (at 115.316 69.596) (size 0.8) (drill 0.4) (layers F.Cu B.Cu) (net 25))
+  (via (at 85.09 80.01) (size 0.8) (drill 0.4) (layers F.Cu B.Cu) (net 25))
+  (via (at 90.17 75.438) (size 0.8) (drill 0.4) (layers F.Cu B.Cu) (net 25))
+  (via (at 103.886 72.39) (size 0.8) (drill 0.4) (layers F.Cu B.Cu) (net 25))
+  (via (at 104.14 77.47) (size 0.8) (drill 0.4) (layers F.Cu B.Cu) (net 25))
+  (via (at 99.06 77.47) (size 0.8) (drill 0.4) (layers F.Cu B.Cu) (net 25))
+  (via (at 92.71 72.898) (size 0.8) (drill 0.4) (layers F.Cu B.Cu) (net 25))
   (segment (start 86.3852 67.324999) (end 86.370201 67.31) (width 0.25) (layer B.Cu) (net 26))
   (segment (start 86.3952 67.334999) (end 86.370201 67.31) (width 1.016) (layer B.Cu) (net 26))
